File: hardware/inverter.brd (EAGLE design)
At the start: 100.3 x 107.6 mm, 51 parts, among them IC1 MEGA8-P, IC2 7805T, K1 ZF112, K2 ZF112, Q5 BC327, Q6 BC327

Commit message: Added gitignore
Parts:
- removed Q10, Q7, Q8, Q9: (no value), transistor:TO92-CBE
- removed R10, R9: (no value), resistor:0207/10
- added R1, R3: (no value), resistor:0207/5V
- added R2, R4: (no value), resistor:0207/2V
- moved Q6 7.62 mm to (86.4, 6.35), turned to 180 degrees
- moved Q5 2.54 mm to (86.4, 39.4), turned to 180 degrees
Connections:
- removed net N$15: Q10.C, Q6.B, Q8.B, R10.1
- removed net N$18: Q5.B, Q7.B, Q9.C, R9.1
- new net N$2: Q6.B, R2.1
- new net N$3: Q5.B, R4.1
- net GND: now also R1.1, R3.1; no longer Q10.E, Q5.C, Q6.C, Q9.E
- net N$13: now also Q6.C, R1.2; no longer Q6.E, Q8.E
- net N$19: now also R2.2; no longer Q10.B
- net N$26: now also Q5.E, Q6.E; no longer Q7.C, Q8.C, R10.2, R9.2
- net N$42: now also R4.2; no longer Q9.B
- net N$6: now also Q5.C, R3.2; no longer Q5.E, Q7.E
Routing:
- net N$18: track 15.2 -> 0.00 mm
- net N$15: track 15.2 -> 0.00 mm
- net N$3: track 0.00 -> 10.2 mm
- net N$2: track 0.00 -> 10.2 mm
- net N$26: track 238.1 -> 233.5 mm
- net N$42: track 9.72 -> 8.45 mm
Changed lines of the file:
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@@
 <attribute name="OC_FARNELL" value="unknown" x="81.28" y="-40.64" size="1.778" layer="27" display="off"/>
 </element>
-<element name="Q5" library="transistor-pnp" package="TO92-EBC" value="BC327" x="86.36" y="36.83"/>
-<element name="Q6" library="transistor-pnp" package="TO92-EBC" value="BC327" x="86.36" y="13.97"/>
-<element name="Q7" library="transistor" package="TO92-CBE" value="" x="86.36" y="40.64"/>
-<element name="Q8" library="transistor" package="TO92-CBE" value="" x="86.36" y="7.62"/>
-<element name="Q9" library="transistor" package="TO92-CBE" value="" x="86.36" y="27.94" rot="R270"/>
-<element name="Q10" library="transistor" package="TO92-CBE" value="" x="86.36" y="20.32" rot="R90"/>
-<element name="R9" library="resistor" package="0207/10" value="" x="81.28" y="38.1" rot="R90"/>
-<element name="R10" library="resistor" package="0207/10" value="" x="81.28" y="10.16" rot="R270"/>
+<element name="Q5" library="transistor-pnp" package="TO92-EBC" value="BC327" x="86.36" y="39.37" rot="R180"/>
+<element name="Q6" library="transistor-pnp" package="TO92-EBC" value="BC327" x="86.36" y="6.35" rot="R180"/>
 <element name="R11" library="resistor" package="0207/5V" value="" x="73.66" y="27.94" rot="R180"/>
 <element name="R12" library="resistor" package="0207/5V" value="" x="73.66" y="20.32" rot="R180"/>
@@
 <element name="R23" library="resistor" package="0207/10" value="" x="78.74" y="10.16" rot="R270"/>
 <element name="D4" library="diode" package="DO15-12" value="1N5060GP" x="17.78" y="35.56"/>
+<element name="R1" library="resistor" package="0207/5V" value="" x="86.36" y="12.7"/>
+<element name="R2" library="resistor" package="0207/2V" value="" x="86.36" y="19.05" rot="R90"/>
+<element name="R3" library="resistor" package="0207/5V" value="" x="86.36" y="35.56"/>
+<element name="R4" library="resistor" package="0207/2V" value="" x="86.36" y="29.21" rot="R270"/>
 </elements>
 <signals>
 <signal name="GND">
 <contactref element="IC1" pad="8"/>
-<contactref element="Q6" pad="C"/>
-<contactref element="Q5" pad="C"/>
-<contactref element="Q9" pad="E"/>
-<contactref element="Q10" pad="E"/>
 <contactref element="Q11" pad="E"/>
 <contactref element="IC2" pad="2"/>
@@
 <contactref element="Q14" pad="E"/>
 <contactref element="D4" pad="A"/>
+<contactref element="R1" pad="1"/>
+<contactref element="R3" pad="1"/>
 </signal>
 <signal name="N$1">
@@
 </signal>
 <signal name="N$13">
-<contactref element="Q6" pad="E"/>
-<contactref element="Q8" pad="E"/>
 <contactref element="JP3" pad="3"/>
-<wire x1="88.9" y1="7.62" x2="88.9" y2="12.7" width="0.6096" layer="16"/>
-<wire x1="88.9" y1="12.7" x2="88.9" y2="20.32" width="0.6096" layer="16"/>
 <wire x1="88.9" y1="20.32" x2="90.17" y2="21.59" width="0.6096" layer="16"/>
 <wire x1="90.17" y1="21.59" x2="92.71" y2="21.59" width="0.6096" layer="16"/>
-</signal>
-<signal name="N$15">
-<contactref element="R10" pad="1"/>
-<contactref element="Q10" pad="C"/>
-<contactref element="Q6" pad="B"/>
-<contactref element="Q8" pad="B"/>
-<wire x1="86.36" y1="7.62" x2="86.36" y2="12.7" width="0.6096" layer="16"/>
-<wire x1="86.36" y1="12.7" x2="86.36" y2="15.24" width="0.6096" layer="16"/>
-<wire x1="86.36" y1="15.24" x2="86.36" y2="17.78" width="0.6096" layer="16"/>
-<wire x1="81.28" y1="15.24" x2="86.36" y2="15.24" width="0.6096" layer="16"/>
-</signal>
-<signal name="N$18">
-<contactref element="R9" pad="1"/>
-<contactref element="Q9" pad="C"/>
-<contactref element="Q5" pad="B"/>
-<contactref element="Q7" pad="B"/>
-<wire x1="86.36" y1="30.48" x2="86.36" y2="33.02" width="0.6096" layer="16"/>
-<wire x1="86.36" y1="33.02" x2="86.36" y2="35.56" width="0.6096" layer="16"/>
-<wire x1="86.36" y1="35.56" x2="86.36" y2="40.64" width="0.6096" layer="16"/>
-<wire x1="81.28" y1="33.02" x2="86.36" y2="33.02" width="0.6096" layer="16"/>
+<contactref element="Q6" pad="C"/>
+<contactref element="R1" pad="2"/>
+<wire x1="88.9" y1="20.32" x2="88.9" y2="12.7" width="0.6096" layer="16"/>
+<wire x1="88.9" y1="11.43" x2="88.9" y2="7.62" width="0.6096" layer="16"/>
+<wire x1="88.9" y1="12.7" x2="88.9" y2="11.43" width="0.6096" layer="16"/>
 </signal>
 <signal name="N$21">
@@
 <contactref element="C3" pad="1"/>
 <contactref element="C1" pad="+"/>
-<contactref element="R10" pad="2"/>
-<contactref element="Q8" pad="C"/>
-<contactref element="R9" pad="2"/>
-<contactref element="Q7" pad="C"/>
 <wire x1="6.35" y1="27.94" x2="6.35" y2="17.78" width="1.27" layer="16"/>
-<wire x1="81.28" y1="43.18" x2="83.82" y2="40.64" width="0.6096" layer="16"/>
-<wire x1="81.28" y1="5.08" x2="83.82" y2="7.62" width="0.6096" layer="16"/>
-<wire x1="83.82" y1="40.64" x2="83.82" y2="43.18" width="1.27" layer="16"/>
 <wire x1="83.82" y1="43.18" x2="85.09" y2="44.45" width="1.27" layer="16"/>
 <wire x1="85.09" y1="44.45" x2="88.9" y2="44.45" width="1.27" layer="16"/>
@@
 <wire x1="92.71" y1="7.62" x2="87.63" y2="2.54" width="1.27" layer="16"/>
 <wire x1="87.63" y1="2.54" x2="83.82" y2="2.54" width="1.27" layer="16"/>
-<wire x1="83.82" y1="2.54" x2="83.82" y2="7.62" width="0.6096" layer="16"/>
-<wire x1="83.82" y1="2.54" x2="73.66" y2="2.54" width="1.27" layer="16"/>
+<wire x1="83.82" y1="2.54" x2="78.74" y2="2.54" width="1.27" layer="16"/>
+<wire x1="78.74" y1="2.54" x2="73.66" y2="2.54" width="1.27" layer="16"/>
 <wire x1="73.66" y1="2.54" x2="48.26" y2="2.54" width="1.27" layer="16"/>
 <wire x1="48.26" y1="2.54" x2="12.7" y2="2.54" width="1.27" layer="16"/>
@@
 <contactref element="R23" pad="2"/>
 <contactref element="R22" pad="2"/>
-<wire x1="78.74" y1="43.18" x2="81.28" y2="43.18" width="0.8128" layer="16"/>
-<wire x1="78.74" y1="5.08" x2="81.28" y2="5.08" width="0.6096" layer="16"/>
+<contactref element="Q6" pad="E"/>
+<wire x1="78.74" y1="5.08" x2="78.74" y2="2.54" width="0.6096" layer="16"/>
+<wire x1="83.82" y1="7.62" x2="83.82" y2="2.54" width="0.6096" layer="16"/>
+<contactref element="Q5" pad="E"/>
+<wire x1="83.82" y1="43.18" x2="83.82" y2="40.64" width="0.8128" layer="16"/>
+<wire x1="78.74" y1="43.18" x2="83.82" y2="43.18" width="0.8128" layer="16"/>
 <wire x1="73.66" y1="2.54" x2="74.93" y2="-26.67" width="0" layer="19" extent="16-16"/>
 </signal>
@@
 <signal name="N$19">
 <contactref element="Q15" pad="C"/>
-<contactref element="Q10" pad="B"/>
 <contactref element="R23" pad="1"/>
 <wire x1="78.74" y1="15.24" x2="81.28" y2="17.78" width="0.6096" layer="16"/>
-<wire x1="86.36" y1="20.32" x2="85.09" y2="20.32" width="0.6096" layer="16"/>
 <wire x1="85.09" y1="20.32" x2="82.55" y2="17.78" width="0.6096" layer="16"/>
 <wire x1="82.55" y1="17.78" x2="81.28" y2="17.78" width="0.6096" layer="16"/>
+<contactref element="R2" pad="2"/>
+<wire x1="85.09" y1="20.32" x2="86.36" y2="20.32" width="0.6096" layer="16"/>
 </signal>
 <signal name="N$20">
@@
 <signal name="N$42">
 <contactref element="Q14" pad="C"/>
-<contactref element="Q9" pad="B"/>
 <contactref element="R22" pad="1"/>
-<wire x1="86.36" y1="27.94" x2="85.09" y2="27.94" width="0.6096" layer="16"/>
 <wire x1="85.09" y1="27.94" x2="82.55" y2="30.48" width="0.6096" layer="16"/>
 <wire x1="82.55" y1="30.48" x2="81.28" y2="30.48" width="0.6096" layer="16"/>
 <wire x1="78.74" y1="33.02" x2="81.28" y2="30.48" width="0.6096" layer="16"/>
+<contactref element="R4" pad="2"/>
+<wire x1="85.09" y1="27.94" x2="86.36" y2="27.94" width="0" layer="19" extent="16-16"/>
 </signal>
 <signal name="N$6">
-<contactref element="Q7" pad="E"/>
-<contactref element="Q5" pad="E"/>
 <contactref element="JP3" pad="1"/>
-<wire x1="88.9" y1="35.56" x2="88.9" y2="27.94" width="0.6096" layer="16"/>
 <wire x1="88.9" y1="27.94" x2="90.17" y2="26.67" width="0.6096" layer="16"/>
 <wire x1="90.17" y1="26.67" x2="92.71" y2="26.67" width="0.6096" layer="16"/>
-<wire x1="88.9" y1="40.64" x2="88.9" y2="35.56" width="0.6096" layer="16"/>
+<contactref element="Q5" pad="C"/>
+<contactref element="R3" pad="2"/>
+<wire x1="88.9" y1="27.94" x2="88.9" y2="35.56" width="0.6096" layer="16"/>
+<wire x1="88.9" y1="35.56" x2="88.9" y2="40.64" width="0.6096" layer="16"/>
+</signal>
+<signal name="N$2">
+<contactref element="R2" pad="1"/>
+<contactref element="Q6" pad="B"/>
+<wire x1="86.36" y1="17.78" x2="86.36" y2="7.62" width="0.6096" layer="16"/>
+</signal>
+<signal name="N$3">
+<contactref element="R4" pad="1"/>
+<contactref element="Q5" pad="B"/>
+<wire x1="86.36" y1="30.48" x2="86.36" y2="40.64" width="0.6096" layer="16"/>
 </signal>
 </signals>
